File: ergogen/routing/proposal/left-trial.kicad_pcb (KiCad board)
At the start: 2 copper layers, 177.3 x 122.5 mm, 130 parts, among them IC1 BQ24075RGTR, IC2 XC6220B331MR-G, J1 USB, J2 BAT, J3 SWD, SW1 RESET, SW2 POWER, Y1 32.768kHz

Commit message: feat(ergogen): move J1 and J2 by hand in the left trial board
J1 to (68.89, 94.6); J2 to (65.5, 114.5), turned from 90 to -90 degrees.
Only the trial board has the moves: left-placed.kicad_pcb still has the
old positions, and the trial's traces still end at the old pads.

Co-Authored-By: Claude Opus 5.5 <noreply@anthropic.com>
Parts:
- moved J2 13.5 mm to (65.5, 114.5), turned to -90 degrees
- moved J1 9.74 mm to (68.9, 94.6)
Changed lines of the file:
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@@
 	(footprint "ogre:USB_PicoEZmate"
 		(layer "B.Cu")
-		(at 78.4952 96.195)
+		(at 68.89 94.6)
 		(property "Reference" "J1"
 			(at 0 -6.95 0)
@@
 	(footprint "ogre:JST_PH_S2B-PH-SM4"
 		(layer "B.Cu")
-		(at 79.0102 114.445 90)
+		(at 65.5 114.5 -90)
 		(property "Reference" "J2"
 			(at 0 -6.925 90)
@@
 		)
 		(fp_line
-			(start 3.95 -3.23)
-			(end 3.95 4.37)
+			(start -3.95 4.37)
+			(end -3.95 -3.23)
 			(stroke
 				(width 0.05)
@@
 		)
 		(fp_line
-			(start 3 -3.23)
-			(end 3.95 -3.23)
+			(start 3.95 4.37)
+			(end -3.95 4.37)
 			(stroke
 				(width 0.05)
@@
 		)
 		(fp_line
-			(start -3 -3.23)
-			(end -3 -1.63)
+			(start -3 -1.63)
+			(end 3 -1.63)
 			(stroke
 				(width 0.05)
@@
 		)
 		(fp_line
-			(start -3.95 -3.23)
-			(end -3 -3.23)
+			(start 3 -1.63)
+			(end 3 -3.23)
 			(stroke
 				(width 0.05)
@@
 		)
 		(fp_line
-			(start 3 -1.63)
-			(end 3 -3.23)
+			(start -3.95 -3.23)
+			(end -3 -3.23)
 			(stroke
 				(width 0.05)
@@
 		)
 		(fp_line
-			(start -3 -1.63)
-			(end 3 -1.63)
+			(start -3 -3.23)
+			(end -3 -1.63)
 			(stroke
 				(width 0.05)
@@
 		)
 		(fp_line
-			(start 3.95 4.37)
-			(end -3.95 4.37)
+			(start 3 -3.23)
+			(end 3.95 -3.23)
 			(stroke
 				(width 0.05)
@@
 		)
 		(fp_line
-			(start -3.95 4.37)
-			(end -3.95 -3.23)
+			(start 3.95 -3.23)
+			(end 3.95 4.37)
 			(stroke
 				(width 0.05)
@@
 		)
 		(fp_line
-			(start 3.95 -3.22)
-			(end 3.95 0.99)
+			(start -2.4 4.37)
+			(end 2.4 4.37)
 			(stroke
 				(width 0.25)
@@
 		)
 		(fp_line
-			(start 3 -3.22)
-			(end 3.95 -3.22)
+			(start -3 -1.65)
+			(end -1.73 -1.65)
 			(stroke
 				(width 0.25)
@@
 		)
 		(fp_line
-			(start -3 -3.22)
-			(end -3 -1.65)
+			(start -0.27 -1.65)
+			(end 0.27 -1.65)
 			(stroke
 				(width 0.25)
@@
 		)
 		(fp_line
-			(start -3.95 -3.22)
-			(end -3 -3.22)
+			(start 1.73 -1.65)
+			(end 3 -1.65)
 			(stroke
 				(width 0.25)
@@
 		)
 		(fp_line
-			(start -3.95 -3.22)
-			(end -3.95 0.99)
+			(start 3 -1.65)
+			(end 3 -3.22)
 			(stroke
 				(width 0.25)
@@
 		)
 		(fp_line
-			(start 3 -1.65)
-			(end 3 -3.22)
+			(start -3.95 -3.22)
+			(end -3.95 0.99)
 			(stroke
 				(width 0.25)
@@
 		)
 		(fp_line
-			(start 1.73 -1.65)
-			(end 3 -1.65)
+			(start -3.95 -3.22)
+			(end -3 -3.22)
 			(stroke
 				(width 0.25)
@@
 		)
 		(fp_line
-			(start -0.27 -1.65)
-			(end 0.27 -1.65)
+			(start -3 -3.22)
+			(end -3 -1.65)
 			(stroke
 				(width 0.25)
@@
 		)
 		(fp_line
-			(start -3 -1.65)
-			(end -1.73 -1.65)
+			(start 3 -3.22)
+			(end 3.95 -3.22)
 			(stroke
 				(width 0.25)
@@
 		)
 		(fp_line
-			(start -2.4 4.37)
-			(end 2.4 4.37)
+			(start 3.95 -3.22)
+			(end 3.95 0.99)
 			(stroke
 				(width 0.25)
@@
 		)
 		(pad "1" smd rect
-			(at 1 -2.93 90)
+			(at 1 -2.93 270)
 			(size 1 3.8)
 			(layers "B.Cu" "B.Mask" "B.Paste")
@@
 		)
 		(pad "2" smd rect
-			(at -1 -2.93 90)
+			(at -1 -2.93 270)
 			(size 1 3.8)
 			(layers "B.Cu" "B.Mask" "B.Paste")
@@
 		)
 		(pad "3" smd rect
-			(at -3.35 2.93 90)
+			(at -3.35 2.93 270)
 			(size 1.5 3.4)
 			(layers "B.Cu" "B.Mask" "B.Paste")
 		)
 		(pad "4" smd rect
-			(at 3.35 2.93 90)
+			(at 3.35 2.93 270)
 			(size 1.5 3.4)
 			(layers "B.Cu" "B.Mask" "B.Paste")
